Commit message: add controller

File: CatModel2_v2_description/urdf/CatModel2_v2.urdf (robot description, URDF)
Before this commit: robot CatModel2_v2, 20 links, 19 joints
Links:
- removed link base_imu
- added link imu_link, mass 0.01; visual box size=0.015 0.015 0.004
Joints:
- removed joint base_imu_joint
- added joint imu_link_joint: type fixed, parent base_link, child imu_link, origin xyz= 0. 0. 0.08 rpy=0. 0. 0.

File: CatModel2_v2_description/xacro/CatModel2_v2.xacro (robot description, xacro)
@@ -2,4 +2,5 @@
 	<xacro:arg name="DEBUG" default="false"/>
   <xacro:include filename="$(find CatModel2_v2_description)/xacro/imu.xacro"/>
+  <xacro:include filename="$(find CatModel2_v2_description)/xacro/ros2_control.xacro"/>
 	<xacro:if value="$(arg DEBUG)">
 		<link name="world"/>
@@ -867,4 +868,4 @@
     <child link="RH_FOOT"/>
   </joint>
-  <xacro:IMU connected_to="base_link" imu_name="base_imu" xyz=" 0.05 0. 0.08" rpy="0. 0. 0."/>
+  <xacro:IMU connected_to="base_link" imu_name="imu_link" xyz=" 0. 0. 0.08" rpy="0. 0. 0."/>
 </robot>

Commit message: fixed_spine

File: CatModel2_v2_description/urdf/CatModel2_v2.urdf (robot description, URDF)
Before this commit: robot CatModel2_v2, 20 links, 19 joints
Joints:
- joint bodyb_yaw_joint: type revolute -> fixed
- joint bodyf_pitch_joint: type revolute -> fixed

File: CatModel2_v2_description/xacro/CatModel2_v2.xacro (robot description, xacro)
@@ -81,5 +81,5 @@
   <joint
     name="bodyf_pitch_joint"
-    type="revolute">
+    type="fixed">
     <origin
       xyz="0 0 0"
@@ -136,5 +136,5 @@
   <joint
     name="bodyb_yaw_joint"
-    type="revolute">
+    type="fixed">
     <origin
       xyz="0 0 0"

File: CatModel2_v2_description/xacro/ros2_control.xacro (robot description, xacro)
@@ -5,14 +5,4 @@
 			<plugin>hardware_CatModel2_mujoco/HardwareCatModel2</plugin>
 		</hardware>
-		<joint name="bodyb_yaw_joint">
-			<command_interface name="position"/>
-			<command_interface name="velocity"/>
-			<command_interface name="effort"/>
-			<command_interface name="kp"/>
-			<command_interface name="kd"/>
-			<state_interface name="position"/>
-			<state_interface name="velocity"/>
-			<state_interface name="effort"/>
-		</joint>
 		<joint name="LH_HAA">
 			<command_interface name="position"/>
@@ -66,14 +56,4 @@
 		</joint>
 		<joint name="RH_KFE">
-			<command_interface name="position"/>
-			<command_interface name="velocity"/>
-			<command_interface name="effort"/>
-			<command_interface name="kp"/>
-			<command_interface name="kd"/>
-			<state_interface name="position"/>
-			<state_interface name="velocity"/>
-			<state_interface name="effort"/>
-		</joint>
-		<joint name="bodyf_pitch_joint">
 			<command_interface name="position"/>
 			<command_interface name="velocity"/>

Commit message: 修改KFE限位

File: CatModel2_v2_description/urdf/CatModel2_v2.urdf (robot description, URDF)
Before this commit: robot CatModel2_v2, 20 links, 19 joints
Joints:
- joint LF_KFE: limit lower=-2.70 upper=-0.92 effort=23.7 velocity=18 -> lower=-2.68 upper=-0.41 effort=23.7 velocity=18
- joint LH_KFE: limit lower=-2.70 upper=-0.92 effort=23.7 velocity=18 -> lower=-2.68 upper=-0.41 effort=23.7 velocity=18
- joint RF_KFE: limit lower=-2.70 upper=-0.92 effort=23.7 velocity=18 -> lower=-2.68 upper=-0.41 effort=23.7 velocity=18
- joint RH_KFE: limit lower=-2.70 upper=-0.92 effort=23.7 velocity=18 -> lower=-2.68 upper=-0.41 effort=23.7 velocity=18

File: CatModel2_v2_description/xacro/CatModel2_v2.xacro (robot description, xacro)
@@ -300,6 +300,6 @@
       xyz="0 1 0" />
     <limit
-      lower="-2.70"
-      upper="-0.92"
+      lower="-2.68"
+      upper="-0.41"
       effort="23.7"
       velocity="18" />
@@ -479,6 +479,6 @@
       xyz="0 1 0" />
     <limit
-      lower="-2.70"
-      upper="-0.92"
+      lower="-2.68"
+      upper="-0.41"
       effort="23.7"
       velocity="18" />
@@ -658,6 +658,6 @@
       xyz="0 1 0" />
     <limit
-      lower="-2.70"
-      upper="-0.92"
+      lower="-2.68"
+      upper="-0.41"
       effort="23.7"
       velocity="18" />
@@ -837,6 +837,6 @@
       xyz="0 1 0" />
     <limit
-      lower="-2.70"
-      upper="-0.92"
+      lower="-2.68"
+      upper="-0.41"
       effort="23.7"
       velocity="18" />

Commit message: 修改力矩限制

File: CatModel2_v2_description/urdf/CatModel2_v2.urdf (robot description, URDF)
Before this commit: robot CatModel2_v2, 20 links, 19 joints
Joints:
- joint LF_HAA: limit lower=-0.785 upper=0.785 effort=23.7 velocity=18 -> lower=-0.785 upper=0.785 effort=23.7 velocity=28.8
- joint LF_HFE: limit lower=-1.05 upper=3.14 effort=23.7 velocity=18 -> lower=-1.05 upper=3.14 effort=23.7 velocity=28.8
- joint LF_KFE: limit lower=-2.70 upper=-0.92 effort=23.7 velocity=18 -> lower=-2.68 upper=-0.41 effort=47.4 velocity=14.4
- joint LH_HAA: limit lower=-0.785 upper=0.785 effort=23.7 velocity=18 -> lower=-0.785 upper=0.785 effort=23.7 velocity=28.8
- joint LH_HFE: limit lower=-1.05 upper=3.14 effort=23.7 velocity=18 -> lower=-1.05 upper=3.14 effort=23.7 velocity=28.8
- joint LH_KFE: limit lower=-2.70 upper=-0.92 effort=23.7 velocity=18 -> lower=-2.68 upper=-0.41 effort=47.4 velocity=14.4
- joint RF_HAA: limit lower=-0.785 upper=0.785 effort=23.7 velocity=18 -> lower=-0.785 upper=0.785 effort=23.7 velocity=28.8
- joint RF_HFE: limit lower=-1.05 upper=3.14 effort=23.7 velocity=18 -> lower=-1.05 upper=3.14 effort=23.7 velocity=28.8
- joint RF_KFE: limit lower=-2.70 upper=-0.92 effort=23.7 velocity=18 -> lower=-2.68 upper=-0.41 effort=47.4 velocity=14.4
- joint RH_HAA: limit lower=-0.785 upper=0.785 effort=23.7 velocity=18 -> lower=-0.785 upper=0.785 effort=23.7 velocity=28.8
- joint RH_HFE: limit lower=-1.05 upper=3.14 effort=23.7 velocity=18 -> lower=-1.05 upper=3.14 effort=23.7 velocity=28.8
- joint RH_KFE: limit lower=-2.70 upper=-0.92 effort=23.7 velocity=18 -> lower=-2.68 upper=-0.41 effort=47.4 velocity=14.4
- joint bodyb_yaw_joint: limit lower=-0.75 upper=0.75 effort=23.7 velocity=18 -> lower=-0.75 upper=0.75 effort=23.7 velocity=28.8
- joint bodyf_pitch_joint: limit lower=-0.75 upper=0.75 effort=23.7 velocity=18 -> lower=-0.75 upper=0.75 effort=23.7 velocity=28.8
- joint imu_link_joint: origin xyz= 0. 0. 0.08 rpy=0. 0. 0. -> xyz= 0. 0. -0.18 rpy=0. 0. 0.

File: CatModel2_v2_description/xacro/CatModel2_v2.xacro (robot description, xacro)
@@ -95,5 +95,5 @@
       upper="0.75"
       effort="23.7"
-      velocity="18" />
+      velocity="28.8" />
   </joint>
     <link
@@ -150,5 +150,5 @@
       upper="0.75"
       effort="23.7"
-      velocity="18" />
+      velocity="28.8" />
   </joint>
   <link
@@ -199,5 +199,5 @@
       upper="0.785"
       effort="23.7"
-      velocity="18" />
+      velocity="28.8" />
   </joint>
   <link
@@ -248,5 +248,5 @@
       upper="3.14"
       effort="23.7"
-      velocity="18" />
+      velocity="28.8" />
   </joint>
   <link
@@ -300,8 +300,8 @@
       xyz="0 1 0" />
     <limit
-      lower="-2.70"
-      upper="-0.92"
-      effort="23.7"
-      velocity="18" />
+      lower="-2.68"
+      upper="-0.41"
+      effort="47.4"
+      velocity="14.4" />
   </joint>
   <link name="LF_FOOT">
@@ -378,5 +378,5 @@
       upper="0.785"
       effort="23.7"
-      velocity="18" />
+      velocity="28.8" />
   </joint>
   <link
@@ -427,5 +427,5 @@
       upper="3.14"
       effort="23.7"
-      velocity="18" />
+      velocity="28.8" />
   </joint>
   <link
@@ -479,8 +479,8 @@
       xyz="0 1 0" />
     <limit
-      lower="-2.70"
-      upper="-0.92"
-      effort="23.7"
-      velocity="18" />
+      lower="-2.68"
+      upper="-0.41"
+      effort="47.4"
+      velocity="14.4" />
   </joint>
   <link name="RF_FOOT">
@@ -557,5 +557,5 @@
       upper="0.785"
       effort="23.7"
-      velocity="18" />
+      velocity="28.8" />
   </joint>
   <link
@@ -606,5 +606,5 @@
       upper="3.14"
       effort="23.7"
-      velocity="18" />
+      velocity="28.8" />
   </joint>
   <link
@@ -658,8 +658,8 @@
       xyz="0 1 0" />
     <limit
-      lower="-2.70"
-      upper="-0.92"
-      effort="23.7"
-      velocity="18" />
+      lower="-2.68"
+      upper="-0.41"
+      effort="47.4"
+      velocity="14.4" />
   </joint>
   <link name="LH_FOOT">
@@ -736,5 +736,5 @@
       upper="0.785"
       effort="23.7"
-      velocity="18" />
+      velocity="28.8" />
   </joint>
   <link
@@ -785,5 +785,5 @@
       upper="3.14"
       effort="23.7"
-      velocity="18" />
+      velocity="28.8" />
   </joint>
   <link
@@ -837,8 +837,8 @@
       xyz="0 1 0" />
     <limit
-      lower="-2.70"
-      upper="-0.92"
-      effort="23.7"
-      velocity="18" />
+      lower="-2.68"
+      upper="-0.41"
+      effort="47.4"
+      velocity="14.4" />
   </joint>
     <link name="RH_FOOT">
@@ -868,4 +868,4 @@
     <child link="RH_FOOT"/>
   </joint>
-  <xacro:IMU connected_to="base_link" imu_name="imu_link" xyz=" 0. 0. 0.08" rpy="0. 0. 0."/>
+  <xacro:IMU connected_to="base_link" imu_name="imu_link" xyz=" 0. 0. -0.18" rpy="0. 0. 0."/>
 </robot>

Commit message: 修改力矩限制

File: CatModel2_v2_description/urdf/CatModel2_v2.urdf (robot description, URDF)
Before this commit: robot CatModel2_v2, 20 links, 19 joints
Joints:
- joint LF_HAA: limit lower=-0.785 upper=0.785 effort=23.7 velocity=18 -> lower=-0.785 upper=0.785 effort=23.7 velocity=28.8
- joint LF_HFE: limit lower=-1.05 upper=3.14 effort=23.7 velocity=18 -> lower=-1.05 upper=3.14 effort=23.7 velocity=28.8
- joint LF_KFE: limit lower=-2.68 upper=-0.41 effort=23.7 velocity=18 -> lower=-2.68 upper=-0.41 effort=47.4 velocity=14.4
- joint LH_HAA: limit lower=-0.785 upper=0.785 effort=23.7 velocity=18 -> lower=-0.785 upper=0.785 effort=23.7 velocity=28.8
- joint LH_HFE: limit lower=-1.05 upper=3.14 effort=23.7 velocity=18 -> lower=-1.05 upper=3.14 effort=23.7 velocity=28.8
- joint LH_KFE: limit lower=-2.68 upper=-0.41 effort=23.7 velocity=18 -> lower=-2.68 upper=-0.41 effort=47.4 velocity=14.4
- joint RF_HAA: limit lower=-0.785 upper=0.785 effort=23.7 velocity=18 -> lower=-0.785 upper=0.785 effort=23.7 velocity=28.8
- joint RF_HFE: limit lower=-1.05 upper=3.14 effort=23.7 velocity=18 -> lower=-1.05 upper=3.14 effort=23.7 velocity=28.8
- joint RF_KFE: limit lower=-2.68 upper=-0.41 effort=23.7 velocity=18 -> lower=-2.68 upper=-0.41 effort=47.4 velocity=14.4
- joint RH_HAA: limit lower=-0.785 upper=0.785 effort=23.7 velocity=18 -> lower=-0.785 upper=0.785 effort=23.7 velocity=28.8
- joint RH_HFE: limit lower=-1.05 upper=3.14 effort=23.7 velocity=18 -> lower=-1.05 upper=3.14 effort=23.7 velocity=28.8
- joint RH_KFE: limit lower=-2.68 upper=-0.41 effort=23.7 velocity=18 -> lower=-2.68 upper=-0.41 effort=47.4 velocity=14.4

File: CatModel2_v2_description/xacro/CatModel2_v2.xacro (robot description, xacro)
@@ -199,5 +199,5 @@
       upper="0.785"
       effort="23.7"
-      velocity="18" />
+      velocity="28.8" />
   </joint>
   <link
@@ -248,5 +248,5 @@
       upper="3.14"
       effort="23.7"
-      velocity="18" />
+      velocity="28.8" />
   </joint>
   <link
@@ -302,6 +302,6 @@
       lower="-2.68"
       upper="-0.41"
-      effort="23.7"
-      velocity="18" />
+      effort="47.4"
+      velocity="14.4" />
   </joint>
   <link name="LF_FOOT">
@@ -378,5 +378,5 @@
       upper="0.785"
       effort="23.7"
-      velocity="18" />
+      velocity="28.8" />
   </joint>
   <link
@@ -427,5 +427,5 @@
       upper="3.14"
       effort="23.7"
-      velocity="18" />
+      velocity="28.8" />
   </joint>
   <link
@@ -481,6 +481,6 @@
       lower="-2.68"
       upper="-0.41"
-      effort="23.7"
-      velocity="18" />
+      effort="47.4"
+      velocity="14.4" />
   </joint>
   <link name="RF_FOOT">
@@ -557,5 +557,5 @@
       upper="0.785"
       effort="23.7"
-      velocity="18" />
+      velocity="28.8" />
   </joint>
   <link
@@ -606,5 +606,5 @@
       upper="3.14"
       effort="23.7"
-      velocity="18" />
+      velocity="28.8" />
   </joint>
   <link
@@ -660,6 +660,6 @@
       lower="-2.68"
       upper="-0.41"
-      effort="23.7"
-      velocity="18" />
+      effort="47.4"
+      velocity="14.4" />
   </joint>
   <link name="LH_FOOT">
@@ -736,5 +736,5 @@
       upper="0.785"
       effort="23.7"
-      velocity="18" />
+      velocity="28.8" />
   </joint>
   <link
@@ -785,5 +785,5 @@
       upper="3.14"
       effort="23.7"
-      velocity="18" />
+      velocity="28.8" />
   </joint>
   <link
@@ -839,6 +839,6 @@
       lower="-2.68"
       upper="-0.41"
-      effort="23.7"
-      velocity="18" />
+      effort="47.4"
+      velocity="14.4" />
   </joint>
     <link name="RH_FOOT">

Commit message: 修改了脊椎关节的位置,参考的关节位置,wbc力矩限制

File: CatModel2_v2_description/urdf/CatModel2_v2.urdf (robot description, URDF)
Before this commit: robot CatModel2_v2, 20 links, 19 joints
Joints:
- joint bodyb_yaw_joint: origin xyz=0 0 0 rpy=0 0 0 -> xyz=-0.015 0 0 rpy=0 0 0
- joint bodyf_pitch_joint: origin xyz=0 0 0 rpy=0 0 0 -> xyz=0.02 0 0 rpy=0 0 0

File: CatModel2_v2_description/xacro/CatModel2_v2.xacro (robot description, xacro)
@@ -83,5 +83,5 @@
     type="revolute">
     <origin
-      xyz="0 0 0"
+      xyz="0.02 0 0"
       rpy="0 0 0" />
     <parent
@@ -138,5 +138,5 @@
     type="revolute">
     <origin
-      xyz="0 0 0"
+      xyz="-0.015 0 0"
       rpy="0 0 0" />
     <parent
