Commit message: 无脊椎新惯量

File: CatModel2_v2_description/urdf/CatModel2_v2.urdf (robot description, URDF)
Before this commit: robot CatModel2_v2, 20 links, 19 joints
Links:
- link BB_Link: mass 3.23275137200683 -> 3.2327577415008
- link BF_Link: mass 3.1773 -> 3.17726715851683
- link LF_calf: mass 0.14476 -> 0.144759009545625
- link LF_hip: mass 0.64023 -> 0.640227659563685
- link LF_thigh: mass 0.90246 -> 0.902429382815121
- link LH_hip: mass 0.64022505148254 -> 0.640227659584975
- link LH_thigh: mass 0.90245513578387 -> 0.902429402319732
- link RF_hip: mass 0.640225051482545 -> 0.640227659563686
- link RF_thigh: mass 0.902455135679806 -> 0.902429400703756
- link RH_hip: mass 0.642366646261419 -> 0.640227659651105
- link base_link: mass 0.29241 -> 0.292406383722703
Joints:
- joint LF_HAA: origin xyz=0.2106 0.05498 -0.00027501 rpy=0 0 0 -> xyz=0.1856 0.05498 0.0056499 rpy=0 0 0
- joint LH_HAA: origin xyz=-0.2306 0.05498 -0.00027501 rpy=0 0 0 -> xyz=-0.2106 0.05498 -0.00027501 rpy=0 0 0
- joint RF_HAA: origin xyz=0.2106 -0.05502 -0.00027501 rpy=0 0 0 -> xyz=0.1856 -0.05502 0.0056499 rpy=0 0 0
- joint RH_HAA: origin xyz=-0.2306 -0.05502 -0.00027501 rpy=0 0 0 -> xyz=-0.2106 -0.05502 -0.00027501 rpy=0 0 0
- joint bodyb_yaw_joint: limit lower=-0.75 upper=0.75 effort=23.7 velocity=18 -> lower=-0.75 upper=0.75 effort=23.7 velocity=28.8; origin xyz=0 0 0 rpy=0 0 0 -> xyz=-0.02 0 0 rpy=0 0 0
- joint bodyf_pitch_joint: limit lower=-0.75 upper=0.75 effort=23.7 velocity=18 -> lower=-0.75 upper=0.75 effort=23.7 velocity=28.8; origin xyz=0 0 0 rpy=0 0 0 -> xyz=0.025 0 -0.0059249 rpy=0 0 0

File: CatModel2_v2_description/xacro/CatModel2_v2.xacro (robot description, xacro)
@@ -11,19 +11,237 @@
 		</joint>
 	</xacro:if>
-  <link
-    name="base_link">
+ <link name="base_link">
+    <inertial>
+      <origin xyz="0.00277323920478635 -0.000683626781969149 0.000994370734501378" rpy="0 0 0" />
+      <mass value="0.292406383722703" />
+      <inertia ixx="0.00068891" ixy="0.0000208" ixz="-0.00000311" iyy="0.00029552" iyz="0.00002205" izz="0.00050294"/>
+    </inertial>
+    <visual>
+      <origin xyz="0 0 0" rpy="0 0 0" />
+      <geometry>
+        <mesh filename="package://CatModel2_v2_description/meshes/base_link.STL" />
+      </geometry>
+      <material name="">
+        <color rgba="0.752941176470588 0.752941176470588 0.752941176470588 1" />
+      </material>
+    </visual>
+  </link>
+  <link name="BF_Link">
+    <inertial>
+      <origin xyz="0.104546659634399 -8.3815686581723E-05 0.00461080163728378" rpy="0 0 0" />
+      <mass value="3.17726715851683" />
+      <inertia ixx="0.01223609" ixy="0.00015361" ixz="-0.00025349" iyy="0.01896068" iyz="0.00002408" izz="0.02400362"/>
+    </inertial>
+    <visual>
+      <origin xyz="0 0 0" rpy="0 0 0" />
+      <geometry>
+        <mesh filename="package://CatModel2_v2_description/meshes/BF_Link.STL" />
+      </geometry>
+      <material name="">
+        <color rgba="0.752941176470588 0.752941176470588 0.752941176470588 1" />
+      </material>
+    </visual>
+    <collision>
+      <origin rpy="0 0 0" xyz="0.13 0 0"/>
+      <geometry>
+        <box size="0.16 0.2 0.12"/>
+      </geometry>
+    </collision>
+  </link>
+  <joint name="bodyf_pitch_joint" type="fixed">
+    <origin xyz="0.025 0 -0.0059249" rpy="0 0 0" />
+    <parent link="base_link" />
+    <child link="BF_Link" />
+    <axis xyz="0 -1 0" />
+    <limit effort="23.7" lower="-0.75" upper="0.75" velocity="28.8"/>
+  </joint>
+  <link name="BB_Link">
     <inertial>
       <origin
-        xyz="0.0027732 -0.00068363 0.00099437"
-        rpy="0 0 0" />
-      <mass
-        value="0.29241" />
-      <inertia
-        ixx="0.00035365"
-        ixy="-9.4553E-08"
-        ixz="3.37E-07"
-        iyy="0.00014633"
-        iyz="4.7012E-07"
-        izz="0.00023997" />
+        xyz="-0.135121078104581 -0.00203711414555835 -0.0035515309194496" rpy="0 0 0" />
+      <mass value="3.2327577415008" />
+      <inertia ixx="0.01332327" ixy="-0.00015743" ixz="0.00064507" iyy="0.01663537" iyz="0.00007687" izz="0.02166595"/>
+    </inertial>
+    <visual>
+      <origin xyz="0 0 0" rpy="0 0 0" />
+      <geometry>
+        <mesh filename="package://CatModel2_v2_description/meshes/BB_Link.STL" />
+      </geometry>
+      <material name="">
+        <color
+          rgba="0.752941176470588 0.752941176470588 0.752941176470588 1" />
+      </material>
+    </visual>
+    <collision>
+      <origin rpy="0 0 0" xyz="-0.13 0 0"/>
+      <geometry>
+        <box size="0.18 0.2 0.12"/>
+      </geometry>
+    </collision>
+  </link>
+  <joint name="bodyb_yaw_joint" type="fixed">
+    <origin xyz="-0.02 0 0" rpy="0 0 0" />
+    <parent link="base_link" />
+    <child link="BB_Link" />
+    <axis xyz="0 0 1" />
+    <limit effort="23.7" lower="-0.75" upper="0.75" velocity="28.8"/>
+  </joint>
+  <link name="LF_hip">
+    <inertial>
+      <origin xyz="0.0591490110411442 0.000487509404874964 5.42936748087162E-05" rpy="0 0 0" />
+      <mass value="0.640227659563685" />
+      <inertia ixx="0.00047481" ixy="-0.00000256" ixz="0.00000072" iyy="0.00085561" iyz="0.00000037" izz="0.00051370"/>
+    </inertial>
+    <visual>
+      <origin xyz="0 0 0" rpy="0 0 0" />
+      <geometry>
+        <mesh filename="package://CatModel2_v2_description/meshes/LF_hip.STL" />
+      </geometry>
+      <material name="">
+        <color rgba="0.752941176470588 0.752941176470588 0.752941176470588 1" />
+      </material>
+    </visual>
+  </link>
+  <joint name="LF_HAA" type="revolute">
+    <origin xyz="0.1856 0.05498 0.0056499" rpy="0 0 0" />
+    <parent link="BF_Link" />
+    <child link="LF_hip" />
+    <axis xyz="1 0 0" />
+    <limit effort="23.7" lower="-0.785" upper="0.785" velocity="28.8"/>
+  </joint>
+  <link name="LF_thigh">
+    <inertial>
+      <origin xyz="-0.00319263255603119 0.0418746682211462 -0.0295109488745784" rpy="0 0 0" />
+      <mass value="0.902429382815121" />
+      <inertia ixx="0.00398244" ixy="0.00005541" ixz="-0.00029231" iyy="0.00422439" iyz="0.00052841" izz="0.00089724"/>
+    </inertial>
+    <visual>
+      <origin xyz="0 0 0" rpy="0 0 0" />
+      <geometry>
+        <mesh filename="package://CatModel2_v2_description/meshes/LF_thigh.STL" />
+      </geometry>
+      <material name="">
+        <color rgba="0.752941176470588 0.752941176470588 0.752941176470588 1" />
+      </material>
+    </visual>
+  </link>
+  <joint name="LF_HFE" type="revolute">
+    <origin xyz="0.065399 0.02005 0" rpy="0 0 0" />
+    <parent link="LF_hip" />
+    <child link="LF_thigh" />
+    <axis xyz="0 1 0" />
+    <limit effort="23.7" lower="-1.05" upper="3.14" velocity="28.8"/>
+  </joint>
+  <link name="LF_calf">
+    <inertial>
+      <origin xyz="5.55111512312578E-16 1.66533453693773E-16 -0.0526579498337892" rpy="0 0 0" />
+      <mass value="0.144759009545625" />
+      <inertia ixx="0.00056050" ixy="0.00000000" ixz="0.00000000" iyy="0.00057453" iyz="0.00000000" izz="0.00003075"/>
+    </inertial>
+    <visual>
+      <origin xyz="0 0 0" rpy="0 0 0" />
+      <geometry>
+        <mesh
+          filename="package://CatModel2_v2_description/meshes/LF_calf.STL" />
+      </geometry>
+      <material name="">
+        <color rgba="0.101960784313725 0.101960784313725 0.101960784313725 1" />
+      </material>
+    </visual>
+    <collision>
+      <origin rpy="0 1.5707963267948966 0" xyz="0.0 0 -0.068"/>
+      <geometry>
+        <box size="0.18 0.02 0.03"/>
+      </geometry>
+    </collision>
+  </link>
+  <joint name="LF_KFE" type="revolute">
+    <origin xyz="0 0.0617 -0.22" rpy="0 0 0" />
+    <parent link="LF_thigh" />
+    <child link="LF_calf" />
+    <axis xyz="0 1 0" />
+    <limit effort="47.4" lower="-2.68" upper="-0.41" velocity="14.4"/>
+  </joint>
+  <link name="LF_FOOT">
+    <visual>
+      <origin rpy="0 0 0" xyz="0 0 0"/>
+      <geometry>
+        <sphere radius="0.01"/>
+      </geometry>
+      <material name="">
+        <color rgba="0.752941176470588 0.752941176470588 0.752941176470588 1"/>
+      </material>
+    </visual>
+    <collision>
+      <origin rpy="0 0 0" xyz="0 0 0"/>
+      <geometry>
+        <sphere radius="0.02"/>
+      </geometry>
+    </collision>
+    <inertial>
+      <mass value="0.06"/>
+      <inertia ixx="9.600000000000001e-06" ixy="0.0" ixz="0.0" iyy="9.600000000000001e-06" iyz="0.0" izz="9.600000000000001e-06"/>
+    </inertial>
+  </link>
+  <joint name="LF_foot_fixed" type="fixed">
+    <origin rpy="0 0 0" xyz="-0.001 0 -0.18"/>
+    <parent link="LF_calf"/>
+    <child link="LF_FOOT"/>
+  </joint>
+  <link name="RF_hip">
+    <inertial>
+      <origin xyz="0.0591490110411442 -0.000487509404874728 -5.42936748088585E-05" rpy="0 0 0" />
+      <mass value="0.640227659563686" />
+      <inertia ixx="0.00047481" ixy="0.00000256" ixz="-0.00000072" iyy="0.00085561" iyz="0.00000037" izz="0.00051370"/>
+    </inertial>
+    <visual>
+      <origin xyz="0 0 0" rpy="0 0 0" />
+      <geometry>
+        <mesh
+          filename="package://CatModel2_v2_description/meshes/RF_hip.STL" />
+      </geometry>
+      <material name="">
+        <color rgba="0.752941176470588 0.752941176470588 0.752941176470588 1" />
+      </material>
+    </visual>
+  </link>
+  <joint name="RF_HAA"
+    type="revolute">
+    <origin xyz="0.1856 -0.05502 0.0056499" rpy="0 0 0" />
+    <parent link="BF_Link" />
+    <child link="RF_hip" />
+    <axis
+      xyz="1 0 0" />
+    <limit effort="23.7" lower="-0.785" upper="0.785" velocity="28.8"/>
+  </joint>
+  <link name="RF_thigh">
+    <inertial>
+      <origin xyz="-0.00317857966332252 -0.041886419364066 -0.0284744095663136" rpy="0 0 0" />
+      <mass value="0.902429400703756" />
+      <inertia ixx="0.00379972" ixy="-0.00005854" ixz="-0.00029335" iyy="0.00405804" iyz="-0.00050925" izz="0.00091445"/>
+    </inertial>
+    <visual>
+      <origin xyz="0 0 0" rpy="0 0 0" />
+      <geometry>
+        <mesh filename="package://CatModel2_v2_description/meshes/RF_thigh.STL" />
+      </geometry>
+      <material name="">
+        <color rgba="0.752941176470588 0.752941176470588 0.752941176470588 1" />
+      </material>
+    </visual>
+  </link>
+  <joint name="RF_HFE" type="revolute">
+    <origin xyz="0.065399 -0.02005 0" rpy="0 0 0" />
+    <parent link="RF_hip" />
+    <child link="RF_thigh" />
+    <axis xyz="0 1 0" />
+    <limit effort="23.7" lower="-1.05" upper="3.14" velocity="28.8"/>
+  </joint>
+  <link name="RF_calf">
+    <inertial>
+      <origin
+        xyz="6.10622663543836E-16 -6.22765727875674E-15 -0.0526579498337945" rpy="0 0 0" />
+      <mass value="0.144759009545624" />
+      <inertia ixx="0.00056050" ixy="0.00000000" ixz="0.00000000" iyy="0.00057453" iyz="0.00000000" izz="0.00003075"/>
     </inertial>
     <visual>
@@ -33,244 +251,5 @@
       <geometry>
         <mesh
-          filename="package://CatModel2_v2_description/meshes/base_link.STL" />
-      </geometry>
-      <material
-        name="">
-        <color
-          rgba="0.752941176470588 0.752941176470588 0.752941176470588 1" />
-      </material>
-    </visual>
-  </link>
-  <link
-    name="BF_Link">
-    <inertial>
-      <origin
-        xyz="0.12955 -8.3804E-05 -0.0013141"
-        rpy="0 0 0" />
-      <mass
-        value="3.1773" />
-      <inertia
-        ixx="0.0048776"
-        ixy="-5.0175E-06"
-        ixz="-2.0519E-06"
-        iyy="0.0043656"
-        iyz="2.0409E-06"
-        izz="0.0063374" />
-    </inertial>
-    <visual>
-      <origin
-        xyz="0 0 0"
-        rpy="0 0 0" />
-      <geometry>
-        <mesh
-          filename="package://CatModel2_v2_description/meshes/BF_Link.STL" />
-      </geometry>
-      <material
-        name="">
-        <color
-          rgba="0.752941176470588 0.752941176470588 0.752941176470588 1" />
-      </material>
-    </visual>
-    <collision>
-      <origin rpy="0 0 0" xyz="0.13 0 0"/>
-      <geometry>
-        <box size="0.16 0.2 0.12"/>
-      </geometry>
-    </collision>
-  </link>
-  <joint
-    name="bodyf_pitch_joint"
-    type="fixed">
-    <origin
-      xyz="0 0 0"
-      rpy="0 0 0" />
-    <parent
-      link="base_link" />
-    <child
-      link="BF_Link" />
-    <axis
-      xyz="0 -1 0" />
-    <limit
-      lower="-0.75"
-      upper="0.75"
-      effort="23.7"
-      velocity="18" />
-  </joint>
-    <link
-    name="BB_Link">
-    <inertial>
-      <origin
-        xyz="-0.155121047880281 -0.00203708989369605 -0.00355151701603064"
-        rpy="0 0 0" />
-      <mass
-        value="3.23275137200683" />
-      <inertia
-        ixx="0.00514719625702028"
-        ixy="1.12565222116179E-06"
-        ixz="-1.95082644973759E-08"
-        iyy="0.00417841726459602"
-        iyz="-4.35796353082797E-06"
-        izz="0.0068065106450055" />
-    </inertial>
-    <visual>
-      <origin
-        xyz="0 0 0"
-        rpy="0 0 0" />
-      <geometry>
-        <mesh
-          filename="package://CatModel2_v2_description/meshes/BB_Link.STL" />
-      </geometry>
-      <material
-        name="">
-        <color
-          rgba="0.752941176470588 0.752941176470588 0.752941176470588 1" />
-      </material>
-    </visual>
-    <collision>
-      <origin rpy="0 0 0" xyz="-0.13 0 0"/>
-      <geometry>
-        <box size="0.18 0.2 0.12"/>
-      </geometry>
-    </collision>
-  </link>
-  <joint
-    name="bodyb_yaw_joint"
-    type="fixed">
-    <origin
-      xyz="0 0 0"
-      rpy="0 0 0" />
-    <parent
-      link="base_link" />
-    <child
-      link="BB_Link" />
-    <axis
-      xyz="0 0 1" />
-    <limit
-      lower="-0.75"
-      upper="0.75"
-      effort="23.7"
-      velocity="18" />
-  </joint>
-  <link
-    name="LF_hip">
-    <inertial>
-      <origin
-        xyz="0.059149 0.00048753 5.429E-05"
-        rpy="0 0 0" />
-      <mass
-        value="0.64023" />
-      <inertia
-        ixx="0.00043421"
-        ixy="-7.3517E-08"
-        ixz="-9.9092E-07"
-        iyy="0.00072036"
-        iyz="6.9084E-08"
-        izz="0.00034295" />
-    </inertial>
-    <visual>
-      <origin
-        xyz="0 0 0"
-        rpy="0 0 0" />
-      <geometry>
-        <mesh
-          filename="package://CatModel2_v2_description/meshes/LF_hip.STL" />
-      </geometry>
-      <material
-        name="">
-        <color
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