Commit message: BF

File: CatModel2_v2_description/urdf/CatModel2_v2.urdf (robot description, URDF)
Before this commit: robot CatModel2_v2, 19 links, 18 joints
Links:
- link LF_calf: mass 0.144759009545625 -> 0.144759009545624
- link LF_thigh: mass 0.902429382815121 -> 0.902429382860773
- link RF_calf: mass 0.144759009545624 -> 0.144759009545625
- link RF_hip: mass 0.640227659563686 -> 0.640227659563685
- link RH_calf: mass 0.144759009545625 -> 0.144759009545624
- link RH_thigh: mass 0.902455135783871 -> 0.902429402336935
Joints:
- joint LF_HAA: origin xyz=0.1856 0.05498 0.0056499 rpy=0 0 0 -> xyz=0.0781 0.055 0.0056492 rpy=0 0 0
- joint RF_HAA: origin xyz=0.1856 -0.05502 0.0056499 rpy=0 0 0 -> xyz=0.0781 -0.055 0.0056492 rpy=0 0 0
- joint bodyb_yaw_joint: origin xyz=-0.02 0 0 rpy=0 0 0 -> xyz=-0.045 0 0.0059249 rpy=0 0 0
- joint bodyf_pitch_joint: axis 0 -1 0 -> 0 1 0; child BF_Link -> base_link; origin xyz=0.025 0 -0.0059249 rpy=0 0 0 -> xyz=-0.1075 1.9935E-05 0 rpy=0 0 0; parent base_link -> BF_Link

File: CatModel2_v2_description/xacro/CatModel2_v2.xacro (robot description, xacro)
@@ -11,62 +11,94 @@
 		</joint>
 	</xacro:if>
-<link name="base_link">
-    <inertial>
-      <origin xyz="0.00277323920478635 -0.000683626781969149 0.000994370734501378" rpy="0 0 0" />
-      <mass value="0.292406383722703" />
+  <link
+    name="BF_Link">
+    <inertial>
+      <origin
+        xyz="-0.0029532330758115 -6.38809162634701E-05 0.00461007468124051"
+        rpy="0 0 0" />
+      <mass
+        value="3.17726715851683" />
+      <inertia ixx="0.01223609" ixy="0.00015361" ixz="-0.00025349" iyy="0.01896068" iyz="0.00002408" izz="0.02400362"/>
+    </inertial>
+    <visual>
+      <origin
+        xyz="0 0 0"
+        rpy="0 0 0" />
+      <geometry>
+        <mesh
+          filename="package://CatModel2_v2_description/meshes/BF_Link.STL" />
+      </geometry>
+      <material
+        name="">
+        <color
+          rgba="0.752941176470588 0.752941176470588 0.752941176470588 1" />
+      </material>
+    </visual>
+    <collision>
+      <origin rpy="0 0 0" xyz="0 0 0"/>
+      <geometry>
+        <box size="0.16 0.2 0.12"/>
+      </geometry>
+    </collision>
+  </link>
+  <link
+    name="base_link">
+    <inertial>
+      <origin
+        xyz="-0.0222267607952137 -0.000683626781969149 0.00691927164285517"
+        rpy="0 0 0" />
+      <mass
+        value="0.292406383722703" />
       <inertia ixx="0.00068891" ixy="0.0000208" ixz="-0.00000311" iyy="0.00029552" iyz="0.00002205" izz="0.00050294"/>
     </inertial>
     <visual>
-      <origin xyz="0 0 0" rpy="0 0 0" />
-      <geometry>
-        <mesh filename="package://CatModel2_v2_description/meshes/base_link.STL" />
-      </geometry>
-      <material name="">
-        <color rgba="0.752941176470588 0.752941176470588 0.752941176470588 1" />
-      </material>
-    </visual>
-  </link>
-  <link name="BF_Link">
-    <inertial>
-      <origin xyz="0.104546659634399 -8.3815686581723E-05 0.00461080163728378" rpy="0 0 0" />
-      <mass value="3.17726715851683" />
-      <inertia ixx="0.01223609" ixy="0.00015361" ixz="-0.00025349" iyy="0.01896068" iyz="0.00002408" izz="0.02400362"/>
-    </inertial>
-    <visual>
-      <origin xyz="0 0 0" rpy="0 0 0" />
-      <geometry>
-        <mesh filename="package://CatModel2_v2_description/meshes/BF_Link.STL" />
-      </geometry>
-      <material name="">
-        <color rgba="0.752941176470588 0.752941176470588 0.752941176470588 1" />
-      </material>
-    </visual>
-    <collision>
-      <origin rpy="0 0 0" xyz="0.13 0 0"/>
-      <geometry>
-        <box size="0.16 0.2 0.12"/>
-      </geometry>
-    </collision>
-  </link>
-  <joint name="bodyf_pitch_joint" type="revolute">
-    <origin xyz="0.025 0 -0.0059249" rpy="0 0 0" />
-    <parent link="base_link" />
-    <child link="BF_Link" />
-    <axis xyz="0 -1 0" />
+      <origin
+        xyz="0 0 0"
+        rpy="0 0 0" />
+      <geometry>
+        <mesh
+          filename="package://CatModel2_v2_description/meshes/base_link.STL" />
+      </geometry>
+      <material
+        name="">
+        <color
+          rgba="0.752941176470588 0.752941176470588 0.752941176470588 1" />
+      </material>
+    </visual>
+  </link>
+  <joint
+    name="bodyf_pitch_joint"
+    type="revolute">
+    <origin
+      xyz="-0.1075 1.9935E-05 0"
+      rpy="0 0 0" />
+    <parent
+      link="BF_Link" />
+    <child
+      link="base_link" />
+    <axis
+      xyz="0 1 0" />
     <limit effort="23.7" lower="-0.75" upper="0.75" velocity="28.8"/>
   </joint>
-  <link name="BB_Link">
-    <inertial>
-      <origin
-        xyz="-0.135121078104581 -0.00203711414555835 -0.0035515309194496" rpy="0 0 0" />
-      <mass value="3.2327577415008" />
+  <link
+    name="BB_Link">
+    <inertial>
+      <origin
+        xyz="-0.135121078104581 -0.00203711414555829 -0.00355153091944961"
+        rpy="0 0 0" />
+      <mass
+        value="3.2327577415008" />
       <inertia ixx="0.01332327" ixy="-0.00015743" ixz="0.00064507" iyy="0.01663537" iyz="0.00007687" izz="0.02166595"/>
     </inertial>
     <visual>
-      <origin xyz="0 0 0" rpy="0 0 0" />
-      <geometry>
-        <mesh filename="package://CatModel2_v2_description/meshes/BB_Link.STL" />
-      </geometry>
-      <material name="">
+      <origin
+        xyz="0 0 0"
+        rpy="0 0 0" />
+      <geometry>
+        <mesh
+          filename="package://CatModel2_v2_description/meshes/BB_Link.STL" />
+      </geometry>
+      <material
+        name="">
         <color
           rgba="0.752941176470588 0.752941176470588 0.752941176470588 1" />
@@ -80,71 +112,118 @@
     </collision>
   </link>
-  <joint name="bodyb_yaw_joint" type="revolute">
-    <origin xyz="-0.02 0 0" rpy="0 0 0" />
-    <parent link="base_link" />
-    <child link="BB_Link" />
-    <axis xyz="0 0 1" />
+  <joint
+    name="bodyb_yaw_joint"
+    type="revolute">
+    <origin
+      xyz="-0.045 0 0.0059249"
+      rpy="0 0 0" />
+    <parent
+      link="base_link" />
+    <child
+      link="BB_Link" />
+    <axis
+      xyz="0 0 1" />
     <limit effort="23.7" lower="-0.75" upper="0.75" velocity="28.8"/>
   </joint>
-  <link name="LF_hip">
-    <inertial>
-      <origin xyz="0.0591490110411442 0.000487509404874964 5.42936748087162E-05" rpy="0 0 0" />
-      <mass value="0.640227659563685" />
+  <link
+    name="LF_hip">
+    <inertial>
+      <origin
+        xyz="0.059149011041144 0.000487509404874797 5.42936748087336E-05"
+        rpy="0 0 0" />
+      <mass
+        value="0.640227659563685" />
       <inertia ixx="0.00047481" ixy="-0.00000256" ixz="0.00000072" iyy="0.00085561" iyz="0.00000037" izz="0.00051370"/>
     </inertial>
     <visual>
-      <origin xyz="0 0 0" rpy="0 0 0" />
-      <geometry>
-        <mesh filename="package://CatModel2_v2_description/meshes/LF_hip.STL" />
-      </geometry>
-      <material name="">
-        <color rgba="0.752941176470588 0.752941176470588 0.752941176470588 1" />
-      </material>
-    </visual>
-  </link>
-  <joint name="LF_HAA" type="revolute">
-    <origin xyz="0.1856 0.05498 0.0056499" rpy="0 0 0" />
-    <parent link="BF_Link" />
-    <child link="LF_hip" />
-    <axis xyz="1 0 0" />
+      <origin
+        xyz="0 0 0"
+        rpy="0 0 0" />
+      <geometry>
+        <mesh
+          filename="package://CatModel2_v2_description/meshes/LF_hip.STL" />
+      </geometry>
+      <material
+        name="">
+        <color
+          rgba="0.752941176470588 0.752941176470588 0.752941176470588 1" />
+      </material>
+    </visual>
+  </link>
+  <joint
+    name="LF_HAA"
+    type="revolute">
+    <origin
+      xyz="0.0781 0.055 0.0056492"
+      rpy="0 0 0" />
+    <parent
+      link="BF_Link" />
+    <child
+      link="LF_hip" />
+    <axis
+      xyz="1 0 0" />
     <limit effort="23.7" lower="-0.785" upper="0.785" velocity="28.8"/>
   </joint>
-  <link name="LF_thigh">
-    <inertial>
-      <origin xyz="-0.00319263255603119 0.0418746682211462 -0.0295109488745784" rpy="0 0 0" />
-      <mass value="0.902429382815121" />
+  <link
+    name="LF_thigh">
+    <inertial>
+      <origin
+        xyz="-0.00319263255467078 0.0418746682198338 -0.0295109488729833"
+        rpy="0 0 0" />
+      <mass
+        value="0.902429382860773" />
       <inertia ixx="0.00398244" ixy="0.00005541" ixz="-0.00029231" iyy="0.00422439" iyz="0.00052841" izz="0.00089724"/>
     </inertial>
     <visual>
-      <origin xyz="0 0 0" rpy="0 0 0" />
-      <geometry>
-        <mesh filename="package://CatModel2_v2_description/meshes/LF_thigh.STL" />
-      </geometry>
-      <material name="">
-        <color rgba="0.752941176470588 0.752941176470588 0.752941176470588 1" />
-      </material>
-    </visual>
-  </link>
-  <joint name="LF_HFE" type="revolute">
-    <origin xyz="0.065399 0.02005 0" rpy="0 0 0" />
-    <parent link="LF_hip" />
-    <child link="LF_thigh" />
-    <axis xyz="0 1 0" />
+      <origin
+        xyz="0 0 0"
+        rpy="0 0 0" />
+      <geometry>
+        <mesh
+          filename="package://CatModel2_v2_description/meshes/LF_thigh.STL" />
+      </geometry>
+      <material
+        name="">
+        <color
+          rgba="0.752941176470588 0.752941176470588 0.752941176470588 1" />
+      </material>
+    </visual>
+  </link>
+  <joint
+    name="LF_HFE"
+    type="revolute">
+    <origin
+      xyz="0.065399 0.02005 0"
+      rpy="0 0 0" />
+    <parent
+      link="LF_hip" />
+    <child
+      link="LF_thigh" />
+    <axis
+      xyz="0 1 0" />
     <limit effort="23.7" lower="-1.05" upper="3.14" velocity="28.8"/>
   </joint>
-  <link name="LF_calf">
-    <inertial>
-      <origin xyz="5.55111512312578E-16 1.66533453693773E-16 -0.0526579498337892" rpy="0 0 0" />
-      <mass value="0.144759009545625" />
+  <link
+    name="LF_calf">
+    <inertial>
+      <origin
+        xyz="5.55111512312578E-16 1.66533453693773E-16 -0.0526579498337892"
+        rpy="0 0 0" />
+      <mass
+        value="0.144759009545624" />
       <inertia ixx="0.00056050" ixy="0.00000000" ixz="0.00000000" iyy="0.00057453" iyz="0.00000000" izz="0.00003075"/>
     </inertial>
     <visual>
-      <origin xyz="0 0 0" rpy="0 0 0" />
+      <origin
+        xyz="0 0 0"
+        rpy="0 0 0" />
       <geometry>
         <mesh
           filename="package://CatModel2_v2_description/meshes/LF_calf.STL" />
       </geometry>
-      <material name="">
-        <color rgba="0.101960784313725 0.101960784313725 0.101960784313725 1" />
+      <material
+        name="">
+        <color
+          rgba="0.101960784313725 0.101960784313725 0.101960784313725 1" />
       </material>
     </visual>
@@ -156,9 +235,16 @@
     </collision>
   </link>
-  <joint name="LF_KFE" type="revolute">
-    <origin xyz="0 0.0617 -0.22" rpy="0 0 0" />
-    <parent link="LF_thigh" />
-    <child link="LF_calf" />
-    <axis xyz="0 1 0" />
+  <joint
+    name="LF_KFE"
+    type="revolute">
+    <origin
+      xyz="0 0.0617 -0.22"
+      rpy="0 0 0" />
+    <parent
+      link="LF_thigh" />
+    <child
+      link="LF_calf" />
+    <axis
+      xyz="0 1 0" />
     <limit effort="47.4" lower="-2.68" upper="-0.41" velocity="14.4"/>
   </joint>
@@ -189,58 +275,90 @@
     <child link="LF_FOOT"/>
   </joint>
-  <link name="RF_hip">
-    <inertial>
-      <origin xyz="0.0591490110411442 -0.000487509404874728 -5.42936748088585E-05" rpy="0 0 0" />
-      <mass value="0.640227659563686" />
+  <link
+    name="RF_hip">
+    <inertial>
+      <origin
+        xyz="0.059149011041144 -0.000487509404874728 -5.42936748088585E-05"
+        rpy="0 0 0" />
+      <mass
+        value="0.640227659563685" />
       <inertia ixx="0.00047481" ixy="0.00000256" ixz="-0.00000072" iyy="0.00085561" iyz="0.00000037" izz="0.00051370"/>
     </inertial>
     <visual>
-      <origin xyz="0 0 0" rpy="0 0 0" />
+      <origin
+        xyz="0 0 0"
+        rpy="0 0 0" />
       <geometry>
         <mesh
           filename="package://CatModel2_v2_description/meshes/RF_hip.STL" />
       </geometry>
-      <material name="">
-        <color rgba="0.752941176470588 0.752941176470588 0.752941176470588 1" />
-      </material>
-    </visual>
-  </link>
-  <joint name="RF_HAA"
-    type="revolute">
-    <origin xyz="0.1856 -0.05502 0.0056499" rpy="0 0 0" />
-    <parent link="BF_Link" />
-    <child link="RF_hip" />
+      <material
+        name="">
+        <color
+          rgba="0.752941176470588 0.752941176470588 0.752941176470588 1" />
+      </material>
+    </visual>
+  </link>
+  <joint
+    name="RF_HAA"
+    type="revolute">
+    <origin
+      xyz="0.0781 -0.055 0.0056492"
+      rpy="0 0 0" />
+    <parent
+      link="BF_Link" />
+    <child
+      link="RF_hip" />
     <axis
       xyz="1 0 0" />
     <limit effort="23.7" lower="-0.785" upper="0.785" velocity="28.8"/>
   </joint>
-  <link name="RF_thigh">
-    <inertial>
-      <origin xyz="-0.00317857966332252 -0.041886419364066 -0.0284744095663136" rpy="0 0 0" />
-      <mass value="0.902429400703756" />
+  <link
+    name="RF_thigh">
+    <inertial>
+      <origin
+        xyz="-0.00317857966332236 -0.041886419364066 -0.0284744095663136"
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
File: CatModel2_v2_description/xacro/ros2_control.xacro (robot description, xacro)
@@ -5,4 +5,74 @@
 			<plugin>hardware_CatModel2_mujoco/HardwareCatModel2</plugin>
 		</hardware>
+		<joint name="LF_HAA">
+			<command_interface name="position"/>
+			<command_interface name="velocity"/>
+			<command_interface name="effort"/>
+			<command_interface name="kp"/>
+			<command_interface name="kd"/>
+			<state_interface name="position"/>
+			<state_interface name="velocity"/>
+			<state_interface name="effort"/>
+		</joint>
+		<joint name="LF_HFE">
+			<command_interface name="position"/>
+			<command_interface name="velocity"/>
+			<command_interface name="effort"/>
+			<command_interface name="kp"/>
+			<command_interface name="kd"/>
+			<state_interface name="position"/>
+			<state_interface name="velocity"/>
+			<state_interface name="effort"/>
+		</joint>
+		<joint name="LF_KFE">
+			<command_interface name="position"/>
+			<command_interface name="velocity"/>
+			<command_interface name="effort"/>
+			<command_interface name="kp"/>
+			<command_interface name="kd"/>
+			<state_interface name="position"/>
+			<state_interface name="velocity"/>
+			<state_interface name="effort"/>
+		</joint>
+		<joint name="RF_HAA">
+			<command_interface name="position"/>
+			<command_interface name="velocity"/>
+			<command_interface name="effort"/>
+			<command_interface name="kp"/>
+			<command_interface name="kd"/>
+			<state_interface name="position"/>
+			<state_interface name="velocity"/>
+			<state_interface name="effort"/>
+		</joint>
+		<joint name="RF_HFE">
+			<command_interface name="position"/>
+			<command_interface name="velocity"/>
+			<command_interface name="effort"/>
+			<command_interface name="kp"/>
+			<command_interface name="kd"/>
+			<state_interface name="position"/>
+			<state_interface name="velocity"/>
+			<state_interface name="effort"/>
+		</joint>
+		<joint name="RF_KFE">
+			<command_interface name="position"/>
+			<command_interface name="velocity"/>
+			<command_interface name="effort"/>
+			<command_interface name="kp"/>
+			<command_interface name="kd"/>
+			<state_interface name="position"/>
+			<state_interface name="velocity"/>
+			<state_interface name="effort"/>
+		</joint>
+		<joint name="bodyf_pitch_joint">
+			<command_interface name="position"/>
+			<command_interface name="velocity"/>
+			<command_interface name="effort"/>
+			<command_interface name="kp"/>
+			<command_interface name="kd"/>
+			<state_interface name="position"/>
+			<state_interface name="velocity"/>
+			<state_interface name="effort"/>
+		</joint>
 		<joint name="bodyb_yaw_joint">
 			<command_interface name="position"/>
@@ -75,74 +145,4 @@
 			<state_interface name="effort"/>
 		</joint>
-		<joint name="bodyf_pitch_joint">
-			<command_interface name="position"/>
-			<command_interface name="velocity"/>
-			<command_interface name="effort"/>
-			<command_interface name="kp"/>
-			<command_interface name="kd"/>
-			<state_interface name="position"/>
-			<state_interface name="velocity"/>
-			<state_interface name="effort"/>
-		</joint>
-		<joint name="LF_HAA">
-			<command_interface name="position"/>
-			<command_interface name="velocity"/>
-			<command_interface name="effort"/>
-			<command_interface name="kp"/>
-			<command_interface name="kd"/>
-			<state_interface name="position"/>
-			<state_interface name="velocity"/>
-			<state_interface name="effort"/>
-		</joint>
-		<joint name="LF_HFE">
-			<command_interface name="position"/>
-			<command_interface name="velocity"/>
-			<command_interface name="effort"/>
-			<command_interface name="kp"/>
-			<command_interface name="kd"/>
-			<state_interface name="position"/>
-			<state_interface name="velocity"/>
-			<state_interface name="effort"/>
-		</joint>
-		<joint name="LF_KFE">
-			<command_interface name="position"/>
-			<command_interface name="velocity"/>
-			<command_interface name="effort"/>
-			<command_interface name="kp"/>
-			<command_interface name="kd"/>
-			<state_interface name="position"/>
-			<state_interface name="velocity"/>
-			<state_interface name="effort"/>
-		</joint>
-		<joint name="RF_HAA">
-			<command_interface name="position"/>
-			<command_interface name="velocity"/>
-			<command_interface name="effort"/>
-			<command_interface name="kp"/>
-			<command_interface name="kd"/>
-			<state_interface name="position"/>
-			<state_interface name="velocity"/>
-			<state_interface name="effort"/>
-		</joint>
-		<joint name="RF_HFE">
-			<command_interface name="position"/>
-			<command_interface name="velocity"/>
-			<command_interface name="effort"/>
-			<command_interface name="kp"/>
-			<command_interface name="kd"/>
-			<state_interface name="position"/>
-			<state_interface name="velocity"/>
-			<state_interface name="effort"/>
-		</joint>
-		<joint name="RF_KFE">
-			<command_interface name="position"/>
-			<command_interface name="velocity"/>
-			<command_interface name="effort"/>
-			<command_interface name="kp"/>
-			<command_interface name="kd"/>
-			<state_interface name="position"/>
-			<state_interface name="velocity"/>
-			<state_interface name="effort"/>
-		</joint>
 		<sensor name="imu_sensor">
 			<state_interface name="orientation.w"/>
@@ -158,8 +158,8 @@
 		</sensor>
 		<sensor name="foot_force">
+			<state_interface name="LF"/>
+			<state_interface name="RF"/>
 			<state_interface name="LH"/>
 			<state_interface name="RH"/>
-			<state_interface name="LF"/>
-			<state_interface name="RF"/>
 		</sensor>
 	</ros2_control>
